File: arduino_pro_micro.kicad_sch (KiCad schematic)
At the start: 16 parts, among them J1 10103594-0001LF, J2 Conn_01x12_Pin, J3 Conn_01x12_Pin, U1 ATMEGA32U4-AU, Y1 ECS-160-18-5PX-GM-TR

Commit message: PCB and fabrication outputs
Parts:
- C1, C2, C3: footprint (none) -> Capacitor_SMD:C_0402_1005Metric_Pad0.74x0.62mm_HandSolder
- J1: footprint 10103594-0001LF:AMPHENOL_10103594-0001LF -> 10103594_0001LF (1):AMPHENOL_10103594-0001LF
- J2, J3: footprint (none) -> Connector_PinHeader_2.54mm:PinHeader_1x12_P2.54mm_Vertical
- PWR1: renamed from PWR; footprint (none) -> LED_SMD:LED_0201_0603Metric_Pad0.64x0.40mm_HandSolder
- R1, R2, R3, R4: footprint (none) -> Resistor_SMD:R_0402_1005Metric_Pad0.72x0.64mm_HandSolder
- RESET1: renamed from RESET; footprint 1825910-6:SW_1825910-6-4 -> 1825910_6:SW_1825910-6-4
- RX1: renamed from RX; footprint (none) -> LED_SMD:LED_0201_0603Metric
- TX1: renamed from TX; footprint (none) -> LED_SMD:LED_0201_0603Metric
- U1: footprint ATMEGA32U4-AU:QFP80P1200X1200X120-44N -> ATMEGA32U4_AU:QFP80P1200X1200X120-44N
- Y1: footprint ECS160185PXGMTR -> KiCad:ECS160185PXGMTR
Connections:
- net +5V is gone; now on net VCC: R1.1, U1.42 (AREF), U1.7 (VBUS)
Changed lines of the file:
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@@
 	(wire
 		(pts
-			(xy 135.89 64.77) (xy 135.89 67.31)
-		)
-		(stroke
-			(width 0)
-			(type default)
-		)
-	)
-	(wire
-		(pts
 			(xy 92.71 147.32) (xy 95.25 147.32)
 		)
@@
 	(wire
 		(pts
+			(xy 135.89 64.77) (xy 135.89 67.31)
+		)
+		(stroke
+			(width 0)
+			(type default)
+		)
+	)
+	(wire
+		(pts
 			(xy 91.44 124.46) (xy 95.25 124.46)
 		)
@@
 	)
 	(symbol
-		(lib_id "power:+5V")
-		(at 135.89 64.77 0)
-		(unit 1)
-		(exclude_from_sim no)
-		(in_bom yes)
-		(on_board yes)
-		(dnp no)
-		(fields_autoplaced yes)
-		(property "Reference" "#PWR05"
-			(at 135.89 68.58 0)
-			(effects
-				(font
-					(size 1.27 1.27)
-				)
-				(hide yes)
-			)
-		)
-		(property "Value" "+5V"
-			(at 135.89 59.69 0)
-			(effects
-				(font
-					(size 1.27 1.27)
-				)
-			)
-		)
-		(property "Footprint" ""
-			(at 135.89 64.77 0)
-			(effects
-				(font
-					(size 1.27 1.27)
-				)
-				(hide yes)
-			)
-		)
-		(property "Datasheet" ""
-			(at 135.89 64.77 0)
-			(effects
-				(font
-					(size 1.27 1.27)
-				)
-				(hide yes)
-			)
-		)
-		(property "Description" "Power symbol creates a global label with name \"+5V\""
-			(at 135.89 64.77 0)
-			(effects
-				(font
-					(size 1.27 1.27)
-				)
-				(hide yes)
-			)
-		)
-		(pin "1"
-		)
-		(instances
-			(project ""
-				(path "/5e91b676-ecc2-4d19-a6ed-52cabb6ade0a"
-					(reference "#PWR05")
-					(unit 1)
-				)
-			)
-		)
-	)
-	(symbol
 		(lib_id "power:GND")
 		(at 166.37 133.35 90)
@@
 		(dnp no)
 		(fields_autoplaced yes)
-		(property "Reference" "TX"
+		(property "Reference" "TX1"
 			(at 97.4725 118.11 0)
 			(effects
@@
 			)
 		)
-		(property "Footprint" ""
+		(property "Footprint" "LED_SMD:LED_0201_0603Metric"
 			(at 99.06 124.46 0)
 			(effects
@@
 			(project ""
 				(path "/5e91b676-ecc2-4d19-a6ed-52cabb6ade0a"
-					(reference "TX")
+					(reference "TX1")
 					(unit 1)
 				)
@@
 			)
 		)
-		(property "Footprint" "ATMEGA32U4-AU:QFP80P1200X1200X120-44N"
+		(property "Footprint" "ATMEGA32U4_AU:QFP80P1200X1200X120-44N"
 			(at 151.13 92.71 0)
 			(effects
@@
 		(dnp no)
 		(fields_autoplaced yes)
-		(property "Reference" "RESET"
+		(property "Reference" "RESET1"
 			(at 118.11 34.29 0)
 			(effects
@@
 			)
 		)
-		(property "Footprint" "1825910-6:SW_1825910-6-4"
+		(property "Footprint" "1825910_6:SW_1825910-6-4"
 			(at 118.11 44.45 0)
 			(effects
@@
 			(project ""
 				(path "/5e91b676-ecc2-4d19-a6ed-52cabb6ade0a"
-					(reference "RESET")
+					(reference "RESET1")
 					(unit 1)
 				)
@@
 	)
 	(symbol
+		(lib_id "power:VCC")
+		(at 135.89 64.77 0)
+		(unit 1)
+		(exclude_from_sim no)
+		(in_bom yes)
+		(on_board yes)
+		(dnp no)
+		(fields_autoplaced yes)
+		(property "Reference" "#PWR05"
+			(at 135.89 68.58 0)
+			(effects
+				(font
+					(size 1.27 1.27)
+				)
+				(hide yes)
+			)
+		)
+		(property "Value" "VCC"
+			(at 135.89 59.69 0)
+			(effects
+				(font
+					(size 1.27 1.27)
+				)
+			)
+		)
+		(property "Footprint" ""
+			(at 135.89 64.77 0)
+			(effects
+				(font
+					(size 1.27 1.27)
+				)
+				(hide yes)
+			)
+		)
+		(property "Datasheet" ""
+			(at 135.89 64.77 0)
+			(effects
+				(font
+					(size 1.27 1.27)
+				)
+				(hide yes)
+			)
+		)
+		(property "Description" "Power symbol creates a global label with name \"VCC\""
+			(at 135.89 64.77 0)
+			(effects
+				(font
+					(size 1.27 1.27)
+				)
+				(hide yes)
+			)
+		)
+		(pin "1"
+		)
+		(instances
+			(project ""
+				(path "/5e91b676-ecc2-4d19-a6ed-52cabb6ade0a"
+					(reference "#PWR05")
+					(unit 1)
+				)
+			)
+		)
+	)
+	(symbol
 		(lib_id "Device:LED")
 		(at 99.06 147.32 0)
@@
 		(dnp no)
 		(fields_autoplaced yes)
-		(property "Reference" "PWR"
+		(property "Reference" "PWR1"
 			(at 97.4725 140.97 0)
 			(effects
@@
 			)
 		)
-		(property "Footprint" ""
+		(property "Footprint" "LED_SMD:LED_0201_0603Metric_Pad0.64x0.40mm_HandSolder"
 			(at 99.06 147.32 0)
 			(effects
@@
 			(project ""
 				(path "/5e91b676-ecc2-4d19-a6ed-52cabb6ade0a"
-					(reference "PWR")
+					(reference "PWR1")
 					(unit 1)
 				)
@@
 			)
 		)
-		(property "Footprint" "ECS160185PXGMTR"
+		(property "Footprint" "KiCad:ECS160185PXGMTR"
 			(at 242.57 176.2 0)
 			(effects
@@
 			)
 		)
-		(property "Footprint" ""
+		(property "Footprint" "Capacitor_SMD:C_0402_1005Metric_Pad0.74x0.62mm_HandSolder"
 			(at 243.84 85.09 0)
 			(effects
@@
 	)
 	(symbol
+		(lib_id "power:VCC")
+		(at 128.27 31.75 0)
+		(unit 1)
+		(exclude_from_sim no)
+		(in_bom yes)
+		(on_board yes)
+		(dnp no)
+		(fields_autoplaced yes)
+		(property "Reference" "#PWR016"
+			(at 128.27 35.56 0)
+			(effects
+				(font
+					(size 1.27 1.27)
+				)
+				(hide yes)
+			)
+		)
+		(property "Value" "VCC"
+			(at 128.27 26.67 0)
+			(effects
+				(font
+					(size 1.27 1.27)
+				)
+			)
+		)
+		(property "Footprint" ""
+			(at 128.27 31.75 0)
+			(effects
+				(font
+					(size 1.27 1.27)
+				)
+				(hide yes)
+			)
+		)
+		(property "Datasheet" ""
+			(at 128.27 31.75 0)
+			(effects
+				(font
+					(size 1.27 1.27)
+				)
+				(hide yes)
+			)
+		)
+		(property "Description" "Power symbol creates a global label with name \"VCC\""
+			(at 128.27 31.75 0)
+			(effects
+				(font
+					(size 1.27 1.27)
+				)
+				(hide yes)
+			)
+		)
+		(pin "1"
+		)
+		(instances
+			(project ""
+				(path "/5e91b676-ecc2-4d19-a6ed-52cabb6ade0a"
+					(reference "#PWR016")
+					(unit 1)
+				)
+			)
+		)
+	)
+	(symbol
 		(lib_id "Device:R_Small_US")
 		(at 88.9 124.46 90)
@@
 			)
 		)
-		(property "Footprint" ""
+		(property "Footprint" "Resistor_SMD:R_0402_1005Metric_Pad0.72x0.64mm_HandSolder"
 			(at 88.9 124.46 0)
 			(effects
@@
 		(dnp no)
 		(fields_autoplaced yes)
-		(property "Reference" "RX"
+		(property "Reference" "RX1"
 			(at 97.4725 129.54 0)
 			(effects
@@
 			)
 		)
-		(property "Footprint" ""
+		(property "Footprint" "LED_SMD:LED_0201_0603Metric"
 			(at 99.06 135.89 0)
 			(effects
@@
 			(project ""
 				(path "/5e91b676-ecc2-4d19-a6ed-52cabb6ade0a"
-					(reference "RX")
+					(reference "RX1")
 					(unit 1)
 				)
@@
 			)
 		)
-		(property "Footprint" ""
+		(property "Footprint" "Capacitor_SMD:C_0402_1005Metric_Pad0.74x0.62mm_HandSolder"
 			(at 233.68 85.09 0)
 			(effects
@@
 	)
 	(symbol
-		(lib_id "power:+5V")
-		(at 128.27 31.75 0)
-		(unit 1)
-		(exclude_from_sim no)
-		(in_bom yes)
-		(on_board yes)
-		(dnp no)
-		(fields_autoplaced yes)
-		(property "Reference" "#PWR018"
-			(at 128.27 35.56 0)
-			(effects
-				(font
-					(size 1.27 1.27)
-				)
-				(hide yes)
-			)
-		)
-		(property "Value" "+5V"
-			(at 128.27 26.67 0)
-			(effects
-				(font
-					(size 1.27 1.27)
-				)
-			)
-		)
-		(property "Footprint" ""
-			(at 128.27 31.75 0)
-			(effects
-				(font
-					(size 1.27 1.27)
-				)
-				(hide yes)
-			)
-		)
-		(property "Datasheet" ""
-			(at 128.27 31.75 0)
-			(effects
-				(font
-					(size 1.27 1.27)
-				)
-				(hide yes)
-			)
-		)
-		(property "Description" "Power symbol creates a global label with name \"+5V\""
-			(at 128.27 31.75 0)
-			(effects
-				(font
-					(size 1.27 1.27)
-				)
-				(hide yes)
-			)
-		)
-		(pin "1"
-		)
-		(instances
-			(project ""
-				(path "/5e91b676-ecc2-4d19-a6ed-52cabb6ade0a"
-					(reference "#PWR018")
-					(unit 1)
-				)
-			)
-		)
-	)
-	(symbol
 		(lib_id "power:GND")
 		(at 223.52 121.92 0)
@@
 			)
 		)
-		(property "Footprint" ""
+		(property "Footprint" "Capacitor_SMD:C_0402_1005Metric_Pad0.74x0.62mm_HandSolder"
 			(at 180.34 128.27 0)
 			(effects
@@
 			)
 		)
-		(property "Footprint" ""
+		(property "Footprint" "Resistor_SMD:R_0402_1005Metric_Pad0.72x0.64mm_HandSolder"
 			(at 128.27 36.83 0)
 			(effects
@@
 			)
 		)
-		(property "Footprint" ""
+		(property "Footprint" "Resistor_SMD:R_0402_1005Metric_Pad0.72x0.64mm_HandSolder"
 			(at 88.9 135.89 0)
 			(effects
@@
 			)
 		)
-		(property "Footprint" ""
+		(property "Footprint" "Connector_PinHeader_2.54mm:PinHeader_1x12_P2.54mm_Vertical"
 			(at 83.82 69.85 0)
 			(effects
@@
 			)
 		)
-		(property "Footprint" ""
+		(property "Footprint" "Connector_PinHeader_2.54mm:PinHeader_1x12_P2.54mm_Vertical"
 			(at 49.53 69.85 0)
 			(effects
@@
 			)
 		)
-		(property "Footprint" ""
+		(property "Footprint" "Resistor_SMD:R_0402_1005Metric_Pad0.72x0.64mm_HandSolder"
 			(at 90.17 147.32 0)
 			(effects
@@
 			)
 		)
-		(property "Footprint" "10103594-0001LF:AMPHENOL_10103594-0001LF"
+		(property "Footprint" "10103594_0001LF (1):AMPHENOL_10103594-0001LF"
 			(at 233.68 119.38 0)
 			(effects
